File: Power.kicad_sch (KiCad schematic)
At the start: 48 parts, among them J2 Charge, J3 Battery, Q1 AO3401A, Q2 AO3400A, Q3 AO3401A, U4 FUSB303BTMX, U5 TPS61089, U6 D3V3XA4B10LP, U7 BQ25895RTW, U8 TPS63001

Commit message: convert to through vias
JLCPCB
Parts:
- L1: value 1.8uH -> 2.2uH
Changed lines of the file:
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@@
 			)
 		)
-		(property "Value" "1.8uH"
+		(property "Value" "2.2uH"
 			(at 107.95 130.683 90)
 			(show_name no)
