File: cryobelt.kicad_sch (KiCad schematic)
At the start: 4 parts

Commit message: Fix more bugs
Other:
- sheet ESP32-S3 ports: added OTG; removed none
- sheet Power ports: added OTG; removed none
Changed lines of the file:
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@@
+	(wire
+		(pts
+			(xy 134.62 99.06) (xy 148.59 99.06)
+		)
+		(stroke
+			(width 0)
+			(type default)
+		)
+	)
 	(wire
 		(pts
@@
 	(wire
 		(pts
-			(xy 134.62 111.76) (xy 148.59 111.76)
+			(xy 134.62 115.57) (xy 148.59 115.57)
 		)
 		(stroke
@@
 	(wire
 		(pts
-			(xy 134.62 101.6) (xy 148.59 101.6)
-		)
-		(stroke
-			(width 0)
-			(type default)
-		)
-	)
-	(wire
-		(pts
-			(xy 134.62 114.3) (xy 148.59 114.3)
-		)
-		(stroke
-			(width 0)
-			(type default)
-		)
-	)
-	(wire
-		(pts
-			(xy 134.62 99.06) (xy 148.59 99.06)
+			(xy 134.62 105.41) (xy 148.59 105.41)
+		)
+		(stroke
+			(width 0)
+			(type default)
+		)
+	)
+	(wire
+		(pts
+			(xy 134.62 118.11) (xy 148.59 118.11)
+		)
+		(stroke
+			(width 0)
+			(type default)
+		)
+	)
+	(wire
+		(pts
+			(xy 134.62 102.87) (xy 148.59 102.87)
 		)
 		(stroke
@@
 	)
 	(sheet
-		(at 148.59 109.22)
+		(at 148.59 113.03)
 		(size 12.7 7.62)
 		(exclude_from_sim no)
@@
 		)
 		(property "Sheetname" "Fan Control"
-			(at 148.59 108.5084 0)
+			(at 148.59 112.3184 0)
 			(show_name no)
 			(do_not_autoplace no)
@@
 		)
 		(property "Sheetfile" "Fan Control.kicad_sch"
-			(at 148.59 117.4246 0)
+			(at 148.59 121.2346 0)
 			(show_name no)
 			(do_not_autoplace no)
@@
 		)
 		(pin "FAN_GATE" input
-			(at 148.59 111.76 180)
+			(at 148.59 115.57 180)
 			(effects
 				(font
@@
 		)
 		(pin "I_FAN" output
-			(at 148.59 114.3 180)
+			(at 148.59 118.11 180)
 			(effects
 				(font
@@
 	(sheet
 		(at 121.92 68.58)
-		(size 12.7 48.26)
+		(size 12.7 52.07)
 		(exclude_from_sim no)
 		(in_bom yes)
@@
 		)
 		(property "Sheetfile" "ESP32-S3.kicad_sch"
-			(at 121.92 117.4246 0)
+			(at 121.92 121.2346 0)
 			(show_name no)
 			(do_not_autoplace no)
@@
 		)
 		(pin "FAN_GATE" input
-			(at 134.62 111.76 0)
+			(at 134.62 115.57 0)
 			(effects
 				(font
@@
 		)
 		(pin "I_FAN" input
-			(at 134.62 114.3 0)
+			(at 134.62 118.11 0)
 			(effects
 				(font
@@
 		)
 		(pin "OUT1" input
+			(at 134.62 102.87 0)
+			(effects
+				(font
+					(size 1.27 1.27)
+				)
+				(justify right)
+			)
+		)
+		(pin "OUT2" input
+			(at 134.62 105.41 0)
+			(effects
+				(font
+					(size 1.27 1.27)
+				)
+				(justify right)
+			)
+		)
+		(pin "OTG" output
 			(at 134.62 99.06 0)
-			(effects
-				(font
-					(size 1.27 1.27)
-				)
-				(justify right)
-			)
-		)
-		(pin "OUT2" input
-			(at 134.62 101.6 0)
 			(effects
 				(font
@@
 	(sheet
 		(at 148.59 68.58)
-		(size 12.7 35.56)
+		(size 12.7 39.37)
 		(exclude_from_sim no)
 		(in_bom yes)
@@
 		)
 		(property "Sheetfile" "Power.kicad_sch"
-			(at 148.59 104.7246 0)
+			(at 148.59 108.5346 0)
 			(show_name no)
 			(do_not_autoplace no)
@@
 		)
 		(pin "OUT1" output
+			(at 148.59 102.87 180)
+			(effects
+				(font
+					(size 1.27 1.27)
+				)
+				(justify left)
+			)
+		)
+		(pin "OUT2" output
+			(at 148.59 105.41 180)
+			(effects
+				(font
+					(size 1.27 1.27)
+				)
+				(justify left)
+			)
+		)
+		(pin "OTG" input
 			(at 148.59 99.06 180)
 			(effects
 				(font
-					(size 1.27 1.27)
-				)
-				(justify left)
-			)
-		)
-		(pin "OUT2" output
-			(at 148.59 101.6 180)
-			(effects
-				(font

Commit message: Finalize routed Cryobelt PCB for fabrication
Other:
- sheet ESP32-S3 ports: added FAN_PWM; removed FAN_GATE
- sheet Fan Control ports: added FAN_PWM; removed FAN_GATE
Changed lines of the file:
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@@
 			)
 		)
-		(pin "FAN_GATE" input
-			(at 148.59 115.57 180)
+		(pin "I_FAN" output
+			(at 148.59 118.11 180)
 			(effects
 				(font
@@
 			)
 		)
-		(pin "I_FAN" output
-			(at 148.59 118.11 180)
+		(pin "FAN_PWM" input
+			(at 148.59 115.57 180)
 			(effects
 				(font
@@
 			)
 		)
-		(pin "FAN_GATE" input
-			(at 134.62 115.57 0)
-			(effects
-				(font
-					(size 1.27 1.27)
-				)
-				(justify right)
-			)
-		)
 		(pin "I_FAN" input
 			(at 134.62 118.11 0)
@@
 			(effects
 				(font
+					(size 1.27 1.27)
+				)
+				(justify right)
+			)
+		)
+		(pin "FAN_PWM" output
+			(at 134.62 115.57 0)
+			(effects
+				(font
