File: ESP32-S3.kicad_sch (KiCad schematic)
At the start: 29 parts, among them J1 Speaker, SW1 Reset, SW2 Boot, SW3 Down, SW4 User, SW5 Up, U1 SHT4x, U2 ESP32-S3-MINI-1, U3 MAX98357A

Commit message: Optimise BOM
Parts:
- C1, C3, C7: LCSC Part # C86012 -> C15849; MPN GRM188R61A105KA61D -> CL10A105KB8NNNC; Manufacturer Murata -> Samsung Electro-Mechanics
- C2, C4, C5: LCSC Part # C60474 -> C1525; MPN CC0402KRX7R7BB104 -> CL05B104KO5NNNC; Manufacturer YAGEO -> Samsung Electro-Mechanics
- C6, C8: LCSC Part # C703114 -> C19702; MPN GRM188R61A106KAALD -> CL10A106KP8NNNC; Manufacturer Murata -> Samsung Electro-Mechanics
- R1, R2: LCSC Part # C98220 -> C25804; MPN RC0603FR-0710KL -> 0603WAF1002T5E; Manufacturer YAGEO -> UNI-ROYAL
Changed lines of the file:
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@@
 			)
 		)
-		(property "Manufacturer" "Murata"
+ (property "Manufacturer" "Samsung Electro-Mechanics"
 			(at 0 0 0)
 			(hide yes)
@@
 			)
 		)
-		(property "MPN" "GRM188R61A105KA61D"
+		(property "MPN" "CL10A105KB8NNNC"
 			(at 0 0 0)
 			(hide yes)
@@
 			)
 		)
-		(property "LCSC Part #" "C86012"
+		(property "LCSC Part #" "C15849"
 			(at 0 0 0)
 			(hide yes)
@@
 			)
 		)
-		(property "Manufacturer" "Murata"
+ (property "Manufacturer" "Samsung Electro-Mechanics"
 			(at 0 0 0)
 			(hide yes)
@@
 			)
 		)
-		(property "MPN" "GRM188R61A106KAALD"
+		(property "MPN" "CL10A106KP8NNNC"
 			(at 0 0 0)
 			(hide yes)
@@
 			)
 		)
-		(property "LCSC Part #" "C703114"
+		(property "LCSC Part #" "C19702"
 			(at 0 0 0)
 			(hide yes)
@@
 			)
 		)
-		(property "Manufacturer" "Murata"
+ (property "Manufacturer" "Samsung Electro-Mechanics"
 			(at 0 0 0)
 			(hide yes)
@@
 			)
 		)
-		(property "MPN" "GRM188R61A105KA61D"
+		(property "MPN" "CL10A105KB8NNNC"
 			(at 0 0 0)
 			(hide yes)
@@
 			)
 		)
-		(property "LCSC Part #" "C86012"
+		(property "LCSC Part #" "C15849"
 			(at 0 0 0)
 			(hide yes)
@@
 			)
 		)
-		(property "Manufacturer" "YAGEO"
+ (property "Manufacturer" "UNI-ROYAL"
 			(at 0 0 0)
 			(hide yes)
@@
 			)
 		)
-		(property "MPN" "RC0603FR-0710KL"
+		(property "MPN" "0603WAF1002T5E"
 			(at 0 0 0)
 			(hide yes)
@@
 			)
 		)
-		(property "LCSC Part #" "C98220"
+		(property "LCSC Part #" "C25804"
 			(at 0 0 0)
 			(hide yes)
@@
 			)
 		)
-		(property "Manufacturer" "Murata"
+ (property "Manufacturer" "Samsung Electro-Mechanics"
 			(at 0 0 0)
 			(hide yes)
@@
 			)
 		)
-		(property "MPN" "GRM188R61A106KAALD"
+		(property "MPN" "CL10A106KP8NNNC"
 			(at 0 0 0)
 			(hide yes)
@@
 			)
 		)
-		(property "LCSC Part #" "C703114"
+		(property "LCSC Part #" "C19702"
 			(at 0 0 0)
 			(hide yes)
@@
 			)
 		)
-		(property "Manufacturer" "YAGEO"
+ (property "Manufacturer" "UNI-ROYAL"
 			(at 0 0 0)
 			(hide yes)
@@
 			)
 		)
-		(property "MPN" "RC0603FR-0710KL"
+		(property "MPN" "0603WAF1002T5E"
 			(at 0 0 0)
 			(hide yes)
@@
 			)
 		)
-		(property "LCSC Part #" "C98220"
+		(property "LCSC Part #" "C25804"
 			(at 0 0 0)
 			(hide yes)
@@
 			)
 		)
-		(property "Manufacturer" "YAGEO"
+ (property "Manufacturer" "Samsung Electro-Mechanics"
 			(at 0 0 0)
 			(hide yes)
@@
 			)
 		)
-		(property "MPN" "CC0402KRX7R7BB104"
+		(property "MPN" "CL05B104KO5NNNC"
 			(at 0 0 0)
 			(hide yes)
@@
 			)
 		)
-		(property "LCSC Part #" "C60474"
+		(property "LCSC Part #" "C1525"
 			(at 0 0 0)
 			(hide yes)
@@
 			)
 		)
-		(property "Manufacturer" "Murata"
+ (property "Manufacturer" "Samsung Electro-Mechanics"
 			(at 0 0 0)
 			(hide yes)
@@
 			)
 		)
-		(property "MPN" "GRM188R61A105KA61D"
+		(property "MPN" "CL10A105KB8NNNC"
 			(at 0 0 0)
 			(hide yes)
@@
 			)
 		)
-		(property "LCSC Part #" "C86012"
+		(property "LCSC Part #" "C15849"
 			(at 0 0 0)
 			(hide yes)
@@
 			)
 		)
-		(property "Manufacturer" "YAGEO"
+ (property "Manufacturer" "Samsung Electro-Mechanics"
 			(at 0 0 0)
 			(hide yes)
@@
 			)
 		)
-		(property "MPN" "CC0402KRX7R7BB104"
+		(property "MPN" "CL05B104KO5NNNC"
 			(at 0 0 0)
 			(hide yes)
@@
 			)
 		)
-		(property "LCSC Part #" "C60474"
+		(property "LCSC Part #" "C1525"
 			(at 0 0 0)
 			(hide yes)
@@
 			)
 		)
-		(property "Manufacturer" "YAGEO"
+ (property "Manufacturer" "Samsung Electro-Mechanics"
 			(at 0 0 0)
 			(hide yes)
@@
 			)
 		)
-		(property "MPN" "CC0402KRX7R7BB104"
+		(property "MPN" "CL05B104KO5NNNC"
 			(at 0 0 0)
 			(hide yes)
@@
 			)
 		)
-		(property "LCSC Part #" "C60474"
+		(property "LCSC Part #" "C1525"
 			(at 0 0 0)
 			(hide yes)
