File: ESP32-S3.kicad_sch (KiCad schematic)
At the start: 29 parts, among them J1 Speaker, SW1 Reset, SW2 Boot, SW3 Down, SW4 User, SW5 Up, U1 SHT4x, U2 ESP32-S3-MINI-1, U3 MAX98357A

Commit message: Optimize Cryobelt JLC assembly parts
Parts:
- SW1, SW2: footprint Button_Switch_SMD:SW_SPST_Omron_B3FS-100xP -> Button_Switch_SMD:SW_Push_1P1T_XKB_TS-1187A; LCSC Part # C271750 -> C318884; MPN B3FS-1000P -> TS-1187A-B-A-B; Manufacturer Omron -> XKB Connection
Changed lines of the file:
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@@
 			)
 		)
-		(property "Footprint" "Button_Switch_SMD:SW_SPST_Omron_B3FS-100xP"
+		(property "Footprint" "Button_Switch_SMD:SW_Push_1P1T_XKB_TS-1187A"
 			(at 26.67 39.37 0)
 			(hide yes)
@@
 			)
 		)
-		(property "Datasheet" ""
+		(property "Datasheet" "https://datasheet.lcsc.com/lcsc/2304140030_XKB-Connectivity-TS-1187A-B-A-B_C318884.pdf"
 			(at 26.67 39.37 0)
 			(hide yes)
@@
 			)
 		)
-		(property "Manufacturer" "Omron"
+		(property "Manufacturer" "XKB Connection"
 			(at 0 0 0)
 			(hide yes)
@@
 			)
 		)
-		(property "MPN" "B3FS-1000P"
+		(property "MPN" "TS-1187A-B-A-B"
 			(at 0 0 0)
 			(hide yes)
@@
 			)
 		)
-		(property "LCSC Part #" "C271750"
+		(property "LCSC Part #" "C318884"
 			(at 0 0 0)
 			(hide yes)
@@
 			)
 		)
-		(property "Footprint" "Button_Switch_SMD:SW_SPST_Omron_B3FS-100xP"
+		(property "Footprint" "Button_Switch_SMD:SW_Push_1P1T_XKB_TS-1187A"
 			(at 46.99 36.83 0)
 			(hide yes)
@@
 			)
 		)
-		(property "Datasheet" ""
+		(property "Datasheet" "https://datasheet.lcsc.com/lcsc/2304140030_XKB-Connectivity-TS-1187A-B-A-B_C318884.pdf"
 			(at 46.99 36.83 0)
 			(hide yes)
@@
 			)
 		)
-		(property "Manufacturer" "Omron"
+		(property "Manufacturer" "XKB Connection"
 			(at 0 0 0)
 			(hide yes)
@@
 			)
 		)
-		(property "MPN" "B3FS-1000P"
+		(property "MPN" "TS-1187A-B-A-B"
 			(at 0 0 0)
 			(hide yes)
@@
 			)
 		)
-		(property "LCSC Part #" "C271750"
+		(property "LCSC Part #" "C318884"
 			(at 0 0 0)
 			(hide yes)
