File: Fan Control.kicad_sch (KiCad schematic)
At the start: 9 parts, among them J4 Battery, Q4 AO3400A, U9 INA180A3

Commit message: Reset PCB
Parts:
- added C31: 1uF, Capacitor_SMD:C_0603_1608Metric, symbol Device:C
- added C32: 10uF, Capacitor_SMD:C_0603_1608Metric, symbol Device:C
- renumbered R28 to R25, R29 to R26, R30 to R27, R31 to R28
Connections:
- net FAN+: now also C31.1, C32.1
- net GND: now also C31.2, C32.2
Other:
- moved on the sheet: C29, C30, R25, R26, U9

Commit message: Fully routed, no DRC errors
tysm Kevin :D
Parts:
- J4: value Battery -> Fan
Changed lines of the file:
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@@
 			)
 		)
-		(property "Value" "Battery"
+		(property "Value" "Fan"
 			(at 149.86 107.9499 0)
 			(show_name no)

Commit message: BQ fixes
i hate my life
Parts:
- renumbered R25 to R22, R26 to R23, R27 to R24, R28 to R25
Changed lines of the file:
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@@
 		(dnp no)
 		(fields_autoplaced yes)
-		(property "Reference" "#PWR087"
+		(property "Reference" "#PWR084"
 			(at 97.79 96.52 0)
 			(hide yes)
@@
 			(project "cryobelt"
 				(path "/8888d943-d12c-4f99-a4ba-a016e272f484/ab28a137-5ca4-49ec-83fd-1c9558542ea3"
-					(reference "#PWR087")
+					(reference "#PWR084")
 					(unit 1)
 				)
@@
 		(in_pos_files yes)
 		(dnp no)
-		(property "Reference" "R28"
+		(property "Reference" "R25"
 			(at 167.64 91.4399 0)
 			(show_name no)
@@
 			(project "cryobelt"
 				(path "/8888d943-d12c-4f99-a4ba-a016e272f484/ab28a137-5ca4-49ec-83fd-1c9558542ea3"
-					(reference "R28")
+					(reference "R25")
 					(unit 1)
 				)
@@
 		(dnp no)
 		(fields_autoplaced yes)
-		(property "Reference" "R25"
+		(property "Reference" "R22"
 			(at 80.01 76.2 90)
 			(show_name no)
@@
 			(project "cryobelt"
 				(path "/8888d943-d12c-4f99-a4ba-a016e272f484/ab28a137-5ca4-49ec-83fd-1c9558542ea3"
-					(reference "R25")
+					(reference "R22")
 					(unit 1)
 				)
@@
 		(dnp no)
 		(fields_autoplaced yes)
-		(property "Reference" "#PWR084"
+		(property "Reference" "#PWR081"
 			(at 67.31 106.68 0)
 			(hide yes)
@@
 			(project "cryobelt"
 				(path "/8888d943-d12c-4f99-a4ba-a016e272f484/ab28a137-5ca4-49ec-83fd-1c9558542ea3"
-					(reference "#PWR084")
+					(reference "#PWR081")
 					(unit 1)
 				)
@@
 		(dnp no)
 		(fields_autoplaced yes)
-		(property "Reference" "#PWR086"
+		(property "Reference" "#PWR083"
 			(at 93.98 92.71 0)
 			(hide yes)
@@
 			(project "cryobelt"
 				(path "/8888d943-d12c-4f99-a4ba-a016e272f484/ab28a137-5ca4-49ec-83fd-1c9558542ea3"
-					(reference "#PWR086")
+					(reference "#PWR083")
 					(unit 1)
 				)
@@
 		(dnp no)
 		(fields_autoplaced yes)
-		(property "Reference" "#PWR082"
+		(property "Reference" "#PWR079"
 			(at 68.58 92.71 0)
 			(hide yes)
@@
 			(project "cryobelt"
 				(path "/8888d943-d12c-4f99-a4ba-a016e272f484/ab28a137-5ca4-49ec-83fd-1c9558542ea3"
-					(reference "#PWR082")
+					(reference "#PWR079")
 					(unit 1)
 				)
@@
 		(dnp no)
 		(fields_autoplaced yes)
-		(property "Reference" "#PWR085"
+		(property "Reference" "#PWR082"
 			(at 80.01 124.46 0)
 			(hide yes)
@@
 			(project "cryobelt"
 				(path "/8888d943-d12c-4f99-a4ba-a016e272f484/ab28a137-5ca4-49ec-83fd-1c9558542ea3"
-					(reference "#PWR085")
+					(reference "#PWR082")
 					(unit 1)
 				)
@@
 		(dnp no)
 		(fields_autoplaced yes)
-		(property "Reference" "#PWR088"
+		(property "Reference" "#PWR085"
 			(at 109.22 96.52 0)
 			(hide yes)
@@
 			(project "cryobelt"
 				(path "/8888d943-d12c-4f99-a4ba-a016e272f484/ab28a137-5ca4-49ec-83fd-1c9558542ea3"
-					(reference "#PWR088")
+					(reference "#PWR085")
 					(unit 1)
 				)
@@
 		(dnp no)
 		(fields_autoplaced yes)
-		(property "Reference" "#PWR090"
+		(property "Reference" "#PWR087"
 			(at 175.26 100.33 0)
 			(hide yes)
@@
 			(project "cryobelt"
 				(path "/8888d943-d12c-4f99-a4ba-a016e272f484/ab28a137-5ca4-49ec-83fd-1c9558542ea3"
-					(reference "#PWR090")
+					(reference "#PWR087")
 					(unit 1)
 				)
@@
 		(dnp no)
 		(fields_autoplaced yes)
-		(property "Reference" "#PWR089"
+		(property "Reference" "#PWR086"
 			(at 165.1 102.87 0)
 			(hide yes)
@@
 			(project "cryobelt"
 				(path "/8888d943-d12c-4f99-a4ba-a016e272f484/ab28a137-5ca4-49ec-83fd-1c9558542ea3"
-					(reference "#PWR089")
+					(reference "#PWR086")
 					(unit 1)
 				)
@@
 		(dnp no)
 		(fields_autoplaced yes)
-		(property "Reference" "#PWR083"
+		(property "Reference" "#PWR080"
 			(at 67.31 86.36 0)
 			(hide yes)
@@
 			(project "cryobelt"
 				(path "/8888d943-d12c-4f99-a4ba-a016e272f484/ab28a137-5ca4-49ec-83fd-1c9558542ea3"
-					(reference "#PWR083")
+					(reference "#PWR080")
 					(unit 1)
 				)
@@
 		(in_pos_files yes)
 		(dnp no)
-		(property "Reference" "R26"
+		(property "Reference" "R23"
 			(at 82.55 105.4099 0)
 			(show_name no)
@@
 			(project "cryobelt"
 				(path "/8888d943-d12c-4f99-a4ba-a016e272f484/ab28a137-5ca4-49ec-83fd-1c9558542ea3"
-					(reference "R26")
+					(reference "R23")
 					(unit 1)
 				)
@@
 		(in_pos_files yes)
 		(dnp no)
-		(property "Reference" "R27"
+		(property "Reference" "R24"
 			(at 160.02 95.25 90)
 			(show_name no)
@@
 			(project "cryobelt"
 				(path "/8888d943-d12c-4f99-a4ba-a016e272f484/ab28a137-5ca4-49ec-83fd-1c9558542ea3"
-					(reference "R27")
-					(unit 1)
-				)
+					(reference "R24")
+					(unit 1)
+				)

Commit message: Fix more bugs
Parts:
- renumbered C29 to C30, C30 to C31, C31 to C32, C32 to C33, R22 to R25, R23 to R26, R24 to R27, R25 to R28
Changed lines of the file:
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@@
 		(dnp no)
 		(fields_autoplaced yes)
-		(property "Reference" "C30"
+		(property "Reference" "C31"
 			(at 83.82 113.0299 0)
 			(show_name no)
@@
 			(project "cryobelt"
 				(path "/8888d943-d12c-4f99-a4ba-a016e272f484/ab28a137-5ca4-49ec-83fd-1c9558542ea3"
-					(reference "C30")
+					(reference "C31")
 					(unit 1)
 				)
@@
 		(dnp no)
 		(fields_autoplaced yes)
-		(property "Reference" "#PWR084"
+		(property "Reference" "#PWR088"
 			(at 97.79 96.52 0)
 			(hide yes)
@@
 			(project "cryobelt"
 				(path "/8888d943-d12c-4f99-a4ba-a016e272f484/ab28a137-5ca4-49ec-83fd-1c9558542ea3"
-					(reference "#PWR084")
+					(reference "#PWR088")
 					(unit 1)
 				)
@@
 		(in_pos_files yes)
 		(dnp no)
-		(property "Reference" "R25"
+		(property "Reference" "R28"
 			(at 167.64 91.4399 0)
 			(show_name no)
@@
 			(project "cryobelt"
 				(path "/8888d943-d12c-4f99-a4ba-a016e272f484/ab28a137-5ca4-49ec-83fd-1c9558542ea3"
-					(reference "R25")
+					(reference "R28")
 					(unit 1)
 				)
@@
 		(dnp no)
 		(fields_autoplaced yes)
-		(property "Reference" "R22"
+		(property "Reference" "R25"
 			(at 80.01 76.2 90)
 			(show_name no)
@@
 			(project "cryobelt"
 				(path "/8888d943-d12c-4f99-a4ba-a016e272f484/ab28a137-5ca4-49ec-83fd-1c9558542ea3"
-					(reference "R22")
+					(reference "R25")
 					(unit 1)
 				)
@@
 		(dnp no)
 		(fields_autoplaced yes)
-		(property "Reference" "#PWR081"
+		(property "Reference" "#PWR085"
 			(at 67.31 106.68 0)
 			(hide yes)
@@
 			(project "cryobelt"
 				(path "/8888d943-d12c-4f99-a4ba-a016e272f484/ab28a137-5ca4-49ec-83fd-1c9558542ea3"
-					(reference "#PWR081")
+					(reference "#PWR085")
 					(unit 1)
 				)
@@
 		(dnp no)
 		(fields_autoplaced yes)
-		(property "Reference" "#PWR083"
+		(property "Reference" "#PWR087"
 			(at 93.98 92.71 0)
 			(hide yes)
@@
 			(project "cryobelt"
 				(path "/8888d943-d12c-4f99-a4ba-a016e272f484/ab28a137-5ca4-49ec-83fd-1c9558542ea3"
-					(reference "#PWR083")
+					(reference "#PWR087")
 					(unit 1)
 				)
@@
 		(dnp no)
 		(fields_autoplaced yes)
-		(property "Reference" "#PWR079"
+		(property "Reference" "#PWR083"
 			(at 68.58 92.71 0)
 			(hide yes)
@@
 			(project "cryobelt"
 				(path "/8888d943-d12c-4f99-a4ba-a016e272f484/ab28a137-5ca4-49ec-83fd-1c9558542ea3"
-					(reference "#PWR079")
+					(reference "#PWR083")
 					(unit 1)
 				)
@@
 		(dnp no)
 		(fields_autoplaced yes)
-		(property "Reference" "#PWR082"
+		(property "Reference" "#PWR086"
 			(at 80.01 124.46 0)
 			(hide yes)
@@
 			(project "cryobelt"
 				(path "/8888d943-d12c-4f99-a4ba-a016e272f484/ab28a137-5ca4-49ec-83fd-1c9558542ea3"
-					(reference "#PWR082")
+					(reference "#PWR086")
 					(unit 1)
 				)
@@
 		(dnp no)
 		(fields_autoplaced yes)
-		(property "Reference" "C32"
+		(property "Reference" "C33"
 			(at 113.03 85.0899 0)
 			(show_name no)
@@
 			(project "cryobelt"
 				(path "/8888d943-d12c-4f99-a4ba-a016e272f484/ab28a137-5ca4-49ec-83fd-1c9558542ea3"
-					(reference "C32")
+					(reference "C33")
 					(unit 1)
 				)
@@
 		(dnp no)
 		(fields_autoplaced yes)
-		(property "Reference" "C29"
+		(property "Reference" "C30"
 			(at 71.12 95.2499 0)
 			(show_name no)
@@
 			(project "cryobelt"
 				(path "/8888d943-d12c-4f99-a4ba-a016e272f484/ab28a137-5ca4-49ec-83fd-1c9558542ea3"
-					(reference "C29")
+					(reference "C30")
 					(unit 1)
 				)
@@
 		(dnp no)
 		(fields_autoplaced yes)
-		(property "Reference" "#PWR085"
+		(property "Reference" "#PWR089"
 			(at 109.22 96.52 0)
 			(hide yes)
@@
 			(project "cryobelt"
 				(path "/8888d943-d12c-4f99-a4ba-a016e272f484/ab28a137-5ca4-49ec-83fd-1c9558542ea3"
-					(reference "#PWR085")
+					(reference "#PWR089")
 					(unit 1)
 				)
@@
 		(dnp no)
 		(fields_autoplaced yes)
-		(property "Reference" "#PWR087"
+		(property "Reference" "#PWR091"
 			(at 175.26 100.33 0)
 			(hide yes)
@@
 			(project "cryobelt"
 				(path "/8888d943-d12c-4f99-a4ba-a016e272f484/ab28a137-5ca4-49ec-83fd-1c9558542ea3"
-					(reference "#PWR087")
+					(reference "#PWR091")
 					(unit 1)
 				)
@@
 		(dnp no)
 		(fields_autoplaced yes)
-		(property "Reference" "#PWR086"
+		(property "Reference" "#PWR090"
 			(at 165.1 102.87 0)
 			(hide yes)
@@
 			(project "cryobelt"
 				(path "/8888d943-d12c-4f99-a4ba-a016e272f484/ab28a137-5ca4-49ec-83fd-1c9558542ea3"
-					(reference "#PWR086")
+					(reference "#PWR090")
 					(unit 1)
 				)
@@
 		(dnp no)
 		(fields_autoplaced yes)
-		(property "Reference" "C31"
+		(property "Reference" "C32"
 			(at 101.6 85.0899 0)
 			(show_name no)
@@
 			(project "cryobelt"
 				(path "/8888d943-d12c-4f99-a4ba-a016e272f484/ab28a137-5ca4-49ec-83fd-1c9558542ea3"
-					(reference "C31")
+					(reference "C32")
 					(unit 1)
 				)
@@
 		(dnp no)
 		(fields_autoplaced yes)
-		(property "Reference" "#PWR080"
+		(property "Reference" "#PWR084"
 			(at 67.31 86.36 0)
 			(hide yes)
@@
 			(project "cryobelt"
 				(path "/8888d943-d12c-4f99-a4ba-a016e272f484/ab28a137-5ca4-49ec-83fd-1c9558542ea3"
-					(reference "#PWR080")
+					(reference "#PWR084")
 					(unit 1)
 				)
@@
 		(in_pos_files yes)
 		(dnp no)
-		(property "Reference" "R23"
+		(property "Reference" "R26"
 			(at 82.55 105.4099 0)
 			(show_name no)
@@
 			(project "cryobelt"
 				(path "/8888d943-d12c-4f99-a4ba-a016e272f484/ab28a137-5ca4-49ec-83fd-1c9558542ea3"
-					(reference "R23")
+					(reference "R26")
 					(unit 1)
 				)
@@
 		(in_pos_files yes)
 		(dnp no)
-		(property "Reference" "R24"
+		(property "Reference" "R27"
 			(at 160.02 95.25 90)
 			(show_name no)
@@
 			(project "cryobelt"
 				(path "/8888d943-d12c-4f99-a4ba-a016e272f484/ab28a137-5ca4-49ec-83fd-1c9558542ea3"
-					(reference "R24")
-					(unit 1)
-				)
+					(reference "R27")
+					(unit 1)
+				)

Commit message: Finalize routed Cryobelt PCB for fabrication
Parts:
- removed J4: Fan, Connector_Wire:SolderWire-0.5sqmm_1x02_P4.6mm_D0.9mm_OD2.1mm, symbol Connector_Generic:Conn_01x02
- removed Q4: AO3400A, Package_TO_SOT_SMD:SOT-23, symbol Transistor_FET:AO3400A
- added J4: Conn_01x03_Pin, Connector_JST:JST_GH_SM03B-GHS-TB_1x03-1MP_P1.25mm_Horizontal, symbol Connector:Conn_01x03_Pin
- added Q4: 2N7002, Package_TO_SOT_SMD:SOT-23, symbol Transistor_FET:2N7002
- C30, C31: LCSC Part # (none) -> C14663; MPN (none) -> CC0603KRX7R9BB104; Manufacturer (none) -> YAGEO
- C32: LCSC Part # (none) -> C77046; MPN (none) -> GRM188R61E105KA12D; Manufacturer (none) -> Murata
- C33: LCSC Part # (none) -> C697423; MPN (none) -> GRT188R61E106ME13D; Manufacturer (none) -> Murata
- R25: LCSC Part # (none) -> C7467249; MPN (none) -> FRM121WFR050TM; Manufacturer (none) -> FOJAN
- R26: LCSC Part # (none) -> C22548; MPN (none) -> RC0603FR-071KL; Manufacturer (none) -> YAGEO
- R27: value 100R -> 1k; LCSC Part # (none) -> C22548; MPN (none) -> RC0603FR-071KL; Manufacturer (none) -> YAGEO
- R28: LCSC Part # (none) -> C14675; MPN (none) -> RC0603FR-07100KL; Manufacturer (none) -> YAGEO
- U9: LCSC Part # (none) -> C122882; MPN (none) -> INA180A3IDBVR; Manufacturer (none) -> Texas Instruments
Connections:
- net FAN_GATE is gone; now on an unnamed net: R27.1
- net GND: now also J4.3 (Pin_3), Q4.2 (S)
- net at R28.2: now also Q4.1 (G); no longer R27.2
- net FAN+ renamed +12V_FAN
- net +12V_FAN: now also J4.1 (Pin_1)
- new net: J4.2 (Pin_2), Q4.3 (D)
- new net FAN_PWM: R27.2

Commit message: Resolve R15 and R25 assembly sourcing
Parts:
- R25: value 0.05R/0.1% -> 0.05R/1%
Changed lines of the file:
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@@
 			)
 		)
-		(property "Value" "0.05R/0.1%"
+		(property "Value" "0.05R/1%"
 			(at 80.01 78.74 90)
 			(show_name no)

Commit message: Optimise BOM
Parts:
- C32: LCSC Part # C77046 -> C15849; MPN GRM188R61E105KA12D -> CL10A105KB8NNNC; Manufacturer Murata -> Samsung Electro-Mechanics
- C33: LCSC Part # C697423 -> C96446; MPN GRT188R61E106ME13D -> CL10A106MA8NRNC; Manufacturer Murata -> Samsung Electro-Mechanics
- R26, R27: LCSC Part # C22548 -> C21190; MPN RC0603FR-071KL -> 0603WAF1001T5E; Manufacturer YAGEO -> UNI-ROYAL
- R28: LCSC Part # C14675 -> C25803; MPN RC0603FR-07100KL -> 0603WAF1003T5E; Manufacturer YAGEO -> UNI-ROYAL
Changed lines of the file:
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@@
 			)
 		)
-		(property "Manufacturer" "YAGEO"
-			(at 0 0 0)
-			(hide yes)
-			(show_name no)
-			(do_not_autoplace no)
-			(effects
-				(font
-					(size 1.27 1.27)
-				)
-			)
-		)
-		(property "MPN" "RC0603FR-07100KL"
-			(at 0 0 0)
-			(hide yes)
-			(show_name no)
-			(do_not_autoplace no)
-			(effects
-				(font
-					(size 1.27 1.27)
-				)
-			)
-		)
-		(property "LCSC Part #" "C14675"
+ (property "Manufacturer" "UNI-ROYAL"
+			(at 0 0 0)
+			(hide yes)
+			(show_name no)
+			(do_not_autoplace no)
+			(effects
+				(font
+					(size 1.27 1.27)
+				)
+			)
+		)
+		(property "MPN" "0603WAF1003T5E"
+			(at 0 0 0)
+			(hide yes)
+			(show_name no)
+			(do_not_autoplace no)
+			(effects
+				(font
+					(size 1.27 1.27)
+				)
+			)
+		)
+		(property "LCSC Part #" "C25803"
 			(at 0 0 0)
 			(hide yes)
@@
 			)
 		)
-		(property "Manufacturer" "YAGEO"
-			(at 0 0 0)
-			(hide yes)
-			(show_name no)
-			(do_not_autoplace no)
-			(effects
-				(font
-					(size 1.27 1.27)
-				)
-			)
-		)
-		(property "MPN" "RC0603FR-071KL"
-			(at 0 0 0)
-			(hide yes)
-			(show_name no)
-			(do_not_autoplace no)
-			(effects
-				(font
-					(size 1.27 1.27)
-				)
-			)
-		)
-		(property "LCSC Part #" "C22548"
+ (property "Manufacturer" "UNI-ROYAL"
+			(at 0 0 0)
+			(hide yes)
+			(show_name no)
+			(do_not_autoplace no)
+			(effects
+				(font
+					(size 1.27 1.27)
+				)
+			)
+		)
+		(property "MPN" "0603WAF1001T5E"
+			(at 0 0 0)
+			(hide yes)
+			(show_name no)
+			(do_not_autoplace no)
+			(effects
+				(font
+					(size 1.27 1.27)
+				)
+			)
+		)
+		(property "LCSC Part #" "C21190"
 			(at 0 0 0)
 			(hide yes)
@@
 			)
 		)
-		(property "Manufacturer" "Murata"
-			(at 0 0 0)
-			(hide yes)
-			(show_name no)
-			(do_not_autoplace no)
-			(effects
-				(font
-					(size 1.27 1.27)
-				)
-			)
-		)
-		(property "MPN" "GRT188R61E106ME13D"
-			(at 0 0 0)
-			(hide yes)
-			(show_name no)
-			(do_not_autoplace no)
-			(effects
-				(font
-					(size 1.27 1.27)
-				)
-			)
-		)
-		(property "LCSC Part #" "C697423"
+ (property "Manufacturer" "Samsung Electro-Mechanics"
+			(at 0 0 0)
+			(hide yes)
+			(show_name no)
+			(do_not_autoplace no)
+			(effects
+				(font
+					(size 1.27 1.27)
+				)
+			)
+		)
+		(property "MPN" "CL10A106MA8NRNC"
+			(at 0 0 0)
+			(hide yes)
+			(show_name no)
+			(do_not_autoplace no)
+			(effects
+				(font
+					(size 1.27 1.27)
+				)
+			)
+		)
+		(property "LCSC Part #" "C96446"
 			(at 0 0 0)
 			(hide yes)
@@
 			)
 		)
-		(property "Manufacturer" "Murata"
-			(at 0 0 0)
-			(hide yes)
-			(show_name no)
-			(do_not_autoplace no)
-			(effects
-				(font
-					(size 1.27 1.27)
-				)
-			)
-		)
-		(property "MPN" "GRM188R61E105KA12D"
-			(at 0 0 0)
-			(hide yes)
-			(show_name no)
-			(do_not_autoplace no)
-			(effects
-				(font
-					(size 1.27 1.27)
-				)
-			)
-		)
-		(property "LCSC Part #" "C77046"
+ (property "Manufacturer" "Samsung Electro-Mechanics"
+			(at 0 0 0)
+			(hide yes)
+			(show_name no)
+			(do_not_autoplace no)
+			(effects
+				(font
+					(size 1.27 1.27)
+				)
+			)
+		)
+		(property "MPN" "CL10A105KB8NNNC"
+			(at 0 0 0)
+			(hide yes)
+			(show_name no)
+			(do_not_autoplace no)
+			(effects
+				(font
+					(size 1.27 1.27)
+				)
+			)
+		)
+		(property "LCSC Part #" "C15849"
 			(at 0 0 0)
 			(hide yes)
@@
 			)
 		)
-		(property "Manufacturer" "YAGEO"
-			(at 0 0 0)
-			(hide yes)
-			(show_name no)
-			(do_not_autoplace no)
-			(effects
-				(font
-					(size 1.27 1.27)
-				)
-			)
-		)
-		(property "MPN" "RC0603FR-071KL"
-			(at 0 0 0)
-			(hide yes)
-			(show_name no)
-			(do_not_autoplace no)
-			(effects
-				(font
-					(size 1.27 1.27)
-				)
-			)
-		)
-		(property "LCSC Part #" "C22548"
-			(at 0 0 0)
-			(hide yes)
+ (property "Manufacturer" "UNI-ROYAL"
+			(at 0 0 0)
+			(hide yes)
+			(show_name no)
+			(do_not_autoplace no)
+			(effects
+				(font
+					(size 1.27 1.27)
+				)
+			)
+		)
+		(property "MPN" "0603WAF1001T5E"
+			(at 0 0 0)
+			(hide yes)
+			(show_name no)
+			(do_not_autoplace no)
+			(effects
+				(font
+					(size 1.27 1.27)
+				)
+			)
+		)
+		(property "LCSC Part #" "C21190"
+			(at 0 0 0)
+			(hide yes)

Commit message: Optimize Cryobelt JLC assembly parts
Parts:
- Q4: LCSC Part # C616191 -> C8545; MPN 2N7002-G -> 2N7002; Manufacturer Microchip Technology -> Jiangsu Changjing Electronics Technology Co. Ltd.
- R25: value 0.05R/1% -> 0.01R/1%; LCSC Part # C7467249 -> C7467248; MPN FRM121WFR050TM -> FRM121WFR010TM
Changed lines of the file:
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@@
 			)
 		)
-		(property "Value" "0.05R/1%"
+		(property "Value" "0.01R/1%"
 			(at 80.01 78.74 90)
 			(show_name no)
@@
 			)
 		)
-		(property "MPN" "FRM121WFR050TM"
-			(at 0 0 0)
-			(hide yes)
-			(show_name no)
-			(do_not_autoplace no)
-			(effects
-				(font
-					(size 1.27 1.27)
-				)
-			)
-		)
-		(property "LCSC Part #" "C7467249"
+		(property "MPN" "FRM121WFR010TM"
+			(at 0 0 0)
+			(hide yes)
+			(show_name no)
+			(do_not_autoplace no)
+			(effects
+				(font
+					(size 1.27 1.27)
+				)
+			)
+		)
+		(property "LCSC Part #" "C7467248"
 			(at 0 0 0)
 			(hide yes)
@@
 			)
 		)
-		(property "Datasheet" "https://www.onsemi.com/pub/Collateral/NDS7002A-D.PDF"
+		(property "Datasheet" "https://www.lcsc.com/datasheet/lcsc_datasheet_2304140030_Jiangsu-Changjing-Electronics-Technology-Co---Ltd--2N7002_C8545.pdf"
 			(at 134.62 114.3 0)
 			(hide yes)
@@
 			)
 		)
-		(property "Manufacturer" "Microchip Technology"
-			(at 0 0 0)
-			(hide yes)
-			(show_name no)
-			(do_not_autoplace no)
-			(effects
-				(font
-					(size 1.27 1.27)
-				)
-			)
-		)
-		(property "MPN" "2N7002-G"
-			(at 0 0 0)
-			(hide yes)
-			(show_name no)
-			(do_not_autoplace no)
-			(effects
-				(font
-					(size 1.27 1.27)
-				)
-			)
-		)
-		(property "LCSC Part #" "C616191"
-			(at 0 0 0)
-			(hide yes)
+ (property "Manufacturer" "Jiangsu Changjing Electronics Technology Co. Ltd."
+			(at 0 0 0)
+			(hide yes)
+			(show_name no)
+			(do_not_autoplace no)
+			(effects
+				(font
+					(size 1.27 1.27)
+				)
+			)
+		)
+		(property "MPN" "2N7002"
+			(at 0 0 0)
+			(hide yes)
+			(show_name no)
+			(do_not_autoplace no)
+			(effects
+				(font
+					(size 1.27 1.27)
+				)
+			)
+		)
+		(property "LCSC Part #" "C8545"
+			(at 0 0 0)
+			(hide yes)
