File: cryobelt.kicad_pcb (KiCad board)
At the start: 4 copper layers, 90 x 50 mm, 100 parts, among them J1 Speaker, J2 Charge, J3 Battery, J4 Conn_01x03_Pin, Q1 AO3401A, Q2 AO3400A, Q3 AO3401A, Q4 2N7002, SW1 Reset, SW2 Boot, SW3 Down, SW4 User, SW5 Up, U1 SHT4x, U2 ESP32-S3-MINI-1, U3 MAX98357A, U4 FUSB303BTMX, U5 TPS61089, U6 D3V3XA4B10LP, U7 BQ25895RTW, U8 TPS63001, U9 INA180A3

Commit message: Correct charger bootstrap and audio mode values
Parts:
- C23: value 4.7nF -> 47nF
- R8: value 715k -> 634k
Changed lines of the file:
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@@
 			)
 		)
-		(property "Value" "4.7nF"
+		(property "Value" "47nF"
 			(at 0 1.43 90)
 			(layer "F.Fab")
@@
 			)
 		)
-		(property "Datasheet" ""
+		(property "Datasheet" "https://www.lcsc.com/product-detail/C53084515.html"
 			(at 0 0 90)
 			(layer "F.Fab")
@@
 			)
 		)
-		(property "Description" "Unpolarized capacitor"
+		(property "Description" "47 nF 50 V X7R bootstrap capacitor"
 			(at 0 0 90)
 			(layer "F.Fab")
@@
 			)
 		)
-		(property "Manufacturer" "YAGEO"
+		(property "Manufacturer" "TORCH"
 			(at 0 0 270)
 			(unlocked yes)
@@
 			)
 		)
-		(property "MPN" "CC0603KRX7R9BB472"
+		(property "MPN" "CC0603X7R50V473KN"
 			(at 0 0 270)
 			(unlocked yes)
@@
 			)
 		)
-		(property "LCSC Part #" "C106218"
+		(property "LCSC Part #" "C53084515"
 			(at 0 0 270)
 			(unlocked yes)
@@
 			)
 		)
-		(property "Value" "715k"
+		(property "Value" "634k"
 			(at 0 1.43 0)
 			(layer "F.Fab")
@@
 			)
 		)
-		(property "Datasheet" ""
+		(property "Datasheet" "https://www.lcsc.com/product-detail/C273753.html"
 			(at 0 0 0)
 			(layer "F.Fab")
@@
 			)
 		)
-		(property "Description" "Resistor"
+		(property "Description" "634 kOhm 1% SD_MODE pull-up for summed-mono selection at 3.3 V"
 			(at 0 0 0)
 			(layer "F.Fab")
@@
 			)
 		)
-		(property "MPN" "RC0603FR-07715KL"
+		(property "MPN" "RC0603FR-07634KL"
 			(at 0 0 0)
 			(unlocked yes)
@@
 			)
 		)
-		(property "LCSC Part #" "C137685"
+		(property "LCSC Part #" "C273753"
 			(at 0 0 0)
 			(unlocked yes)

Commit message: Optimize Cryobelt JLC assembly parts
Parts:
- D5: value SS12 -> SS14
- L1, L3: footprint Cryobelt:FEXU0420 -> Inductor_SMD:L_Changjiang_FNR4030S
- L2: footprint Inductor_SMD:L_APV_ANR4020 -> Inductor_SMD:L_Changjiang_FNR4030S
- R11: value 301k -> 300k
- R13: value 270k -> 300k
- R22: value 30.1k -> 30k
- R25: value 0.05R/1% -> 0.01R/1%
- SW1, SW2: footprint Button_Switch_SMD:SW_SPST_Omron_B3FS-100xP -> Button_Switch_SMD:SW_Push_1P1T_XKB_TS-1187A
Routing:
- net GND: track 144.7 -> 138.7 mm, vias 88 -> 84
- net /ESP32-S3/EN: track 20.5 -> 17.8 mm
- net /Power/SW: track 11.2 -> 12.1 mm
- net /ESP32-S3/IO0: track 35.7 -> 36.6 mm
- net +BATT: track 13.8 -> 14.5 mm
